File: pcb/right.kicad_sch (KiCad schematic)
At the start: 25 parts, among them J1 Conn_01x04_Pin, SW1 SW_Push_45deg, SW10 SW_Push_45deg, SW11 SW_Push_45deg, SW12 SW_Push_45deg, SW13 SW_Push_45deg, SW14 SW_Push_45deg, SW15 SW_Push_45deg, SW16 SW_Push_45deg, SW17 SW_Push_45deg, SW18 SW_Push_45deg, SW19 SW_Push_45deg, SW2 SW_Push_45deg, SW3 SW_Push_45deg, SW39 SW_Push_45deg, SW4 SW_Push_45deg, SW5 SW_Push_45deg, SW6 SW_Push_45deg, SW7 SW_Push_45deg, SW8 SW_Push_45deg, SW9 SW_Push_45deg, U1 HOLYIOT-18010-NRF52840

Commit message: add step
Parts:
- removed BT1: Battery_Cell, takemo:MY-1632-03, symbol takemo:Battery_Cell
- removed D1: LED, takemo:LED_0402_1005Metric_Pad0.77x0.64mm_HandSolder, symbol takemo:LED
- removed J1: Conn_01x04_Pin, takemo:PinHeader_1x04_P1.00mm_Vertical, symbol takemo:Conn_01x04_Pin
- removed R1: 1K, takemo:R_0402_1005Metric_Pad0.72x0.64mm_HandSolder, symbol takemo:R
- removed SW1, SW10, SW11, SW12, SW13, SW14, SW15, SW16, SW17, SW18, SW19, SW2, SW3, SW4, SW5, SW6, SW7, SW8, SW9: SW_Push_45deg, takemo:CPG1316S01D02, symbol takemo:SW_Push_45deg
- removed SW39: SW_Push_45deg, takemo:SW_SPST_TS-1088-xR025, symbol takemo:SW_Push_45deg
- removed U1: HOLYIOT-18010-NRF52840, takemo:Holyiot_YJ-18010, symbol takemo:HOLYIOT-18010-NRF52840
- added BT2: Battery_Cell, takemo:MY-1632-03, symbol takemo:Battery_Cell
- added D2: LED, takemo:LED_0402_1005Metric_Pad0.77x0.64mm_HandSolder, symbol takemo:LED
- added J2: Conn_01x04_Pin, takemo:PinHeader_1x04_P1.00mm_Vertical, symbol takemo:Conn_01x04_Pin
- added R2: 1K, takemo:R_0402_1005Metric_Pad0.72x0.64mm_HandSolder, symbol takemo:R
- added SW20, SW21, SW22, SW23, SW24, SW25, SW26, SW27, SW28, SW29, SW30, SW31, SW32, SW33, SW34, SW35, SW36, SW37, SW38: SW_Push_45deg, takemo:CPG1316S01D02, symbol takemo:SW_Push_45deg
- added SW40: SW_Push_45deg, takemo:SW_SPST_TS-1088-xR025, symbol takemo:SW_Push_45deg
- added U2: HOLYIOT-18010-NRF52840, takemo:Holyiot_YJ-18010, symbol takemo:HOLYIOT-18010-NRF52840
Connections:
- net GND: now also BT2.2 (-), J2.4 (Pin_4), R2.2, SW20.2, SW21.2, SW22.2, SW23.2, SW24.2, SW25.2, SW26.2, SW27.2, SW28.2, SW29.2, SW30.2, SW31.2, SW32.2, SW33.2, SW34.2, SW35.2, SW36.2, SW37.2, SW38.2, SW40.2, U2.1 (GND), U2.25 (GND), U2.37 (GND)
- net LED: now also D2.2 (A), U2.3 (P1.10)
- net R1C1: now also SW21.1, U2.15 (P0.07)
- net R1C2: now also SW24.1, U2.16 (P1.09)
- net R1C3: now also SW30.1, U2.17 (P0.12)
- net R1C4: now also SW31.1, U2.18 (P0.23)
- net R1C5: now also SW35.1, U2.19 (P0.21)
- net R2C1: now also SW22.1, U2.26 (P0.22)
- net R2C2: now also SW25.1, U2.27 (P1.00)
- net R2C3: now also SW27.1, U2.28 (P1.03)
- net R2C4: now also SW32.1, U2.29 (P1.01)
- net R2C5: now also SW36.1, U2.30 (P1.02)
- net R3C0: now also SW20.1, U2.13 (P0.05/AIN3)
- net R3C1: now also SW23.1, U2.12 (P0.04/AIN2)
- net R3C2: now also SW26.1, U2.11 (P0.31/AIN7)
- net R3C3: now also SW28.1, U2.10 (P0.30/AIN6)
- net R3C4: now also SW33.1, U2.9 (P0.29/AIN5)
- net R3C5: now also SW37.1, U2.8 (P0.28/AIN4)
- net R4C3: now also SW29.1, U2.4 (P1.13)
- net R4C4: now also SW34.1, U2.5 (P1.15)
- net R4C5: now also SW38.1, U2.6 (P0.03/AIN1)
- net RESET: now also SW40.1, U2.21 (P0.18/RESET)
- net SWC: now also J2.3 (Pin_3), U2.31 (SWDCLK)
- net SWD: now also J2.2 (Pin_2), U2.32 (SWDIO)
- net VBUS: now also BT2.1 (+), U2.22 (VBUS)
- net nRF_VDD: now also J2.1 (Pin_1), U2.14 (VDD)
- new net: D2.1 (K), R2.1
